File: Fugu2-esp32s3-wroom-head.kicad_pcb (KiCad board)
At the start: 2 copper layers, 26 x 23.7 mm, 19 parts, among them J1 Conn_02x03_ESP_PROG, J2 Conn_02x07_Odd_Even, P1 USB4105-GF-A, SW1 SW_Push, U1 ESP32-S3-WROOM-1, U2 TLV70233_SOT23-5

Commit message: fix button
Parts:
- P1: value USB4105-GF-A -> QTGM027; footprint Connector_USB:USB_C_Receptacle_GCT_USB4110 -> open-pe:USB_C_Receptacle_GCT_USB4110
- SW1: value SW_Push -> TS-1088-AR02016; footprint Button_Switch_SMD:SW_SPST_B3U-1000P -> Button_Switch_SMD:SW_Push_SPST_NO_Alps_SKRK
- moved SW1 1.54 mm to (102.3, 59.4), turned to 180 degrees
Routing:
- net USB_D-: track 15.5 -> 20.2 mm
- net RX: track 20.9 -> 22.7 mm
- net USB_D+: track 13.3 -> 14.6 mm
- net GND: track 34.1 -> 33.0 mm
- net IO0: track 20.5 -> 21.4 mm, vias 1 -> 0
