File: Fugu2-esp32s3-wroom-head.kicad_pcb (KiCad board)
At the start: 2 copper layers, 26 x 23.7 mm, 20 parts, among them J1 Conn_02x03_ESP_PROG, J2 Conn_02x07_Odd_Even, P1 QTGM027, SW1 TS-1088-AR02016, U1 ESP32-S3-WROOM-1, U2 TLV70233_SOT23-5

Commit message: bump kicad version
Parts:
- removed REF**: SOT-583-8, Package_TO_SOT_SMD:SOT-583-8

Commit message: up
Parts:
- moved R3 0.49 mm to (97.0, 40.1)
- moved R4 0.26 mm to (97.0, 41.4)
Changed lines of the file:
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@@
 	(footprint "Resistor_SMD:R_0402_1005Metric"
 		(layer "F.Cu")
-		(at 96.9752 40.5892 180)
+		(at 96.9752 40.1 180)
 		(descr "Resistor SMD 0402 (1005 Metric), square (rectangular) end terminal, IPC_7351 nominal, (Body size source: IPC-SM-782 page 72, https://www.pcb-3d.com/wordpress/wp-content/uploads/ipc-sm-782a_amendment_1_and_2.pdf), generated with kicad-footprint-generator")
 		(tags "resistor")
@@
 	(footprint "Resistor_SMD:R_0402_1005Metric"
 		(layer "F.Cu")
-		(at 96.9772 41.656 180)
+		(at 96.9772 41.4 180)
 		(descr "Resistor SMD 0402 (1005 Metric), square (rectangular) end terminal, IPC_7351 nominal, (Body size source: IPC-SM-782 page 72, https://www.pcb-3d.com/wordpress/wp-content/uploads/ipc-sm-782a_amendment_1_and_2.pdf), generated with kicad-footprint-generator")
 		(tags "resistor")
@@
 	)
 	(segment
-		(start 97.4852 39.878)
+		(start 97.4852 39.4148)
 		(end 97.4852 40.5892)
 		(width 0.2)
@@
 		(net 41)
 	)
+	(segment
+		(start 97.5 39.4)
+		(end 97.4852 39.4148)
+		(width 0.2)
+		(layer "F.Cu")
+		(net 41)
+	)
 	(via
-		(at 97.4852 39.878)
+		(at 97.5 39.4)
 		(size 0.6)
 		(drill 0.3)
