File: Fugu2-esp32s3-wroom-head.kicad_sch (KiCad schematic)
At the start: 20 parts, among them J1 Conn_02x03_ESP_PROG, J2 Conn_02x07_Odd_Even, P1 QTGM027, SW1 TS-1088-AR02016, U1 ESP32-S3-WROOM-1, U2 TLV70233_SOT23-5

Commit message: fix button
Parts:
- P1: footprint Connector_USB:USB_C_Receptacle_GCT_USB4110 -> open-pe:USB_C_Receptacle_GCT_USB4110
- SW1: footprint Button_Switch_SMD:SW_SPST_B3U-1000P -> Button_Switch_SMD:SW_Push_SPST_NO_Alps_SKRK; Footprint_alt (none) -> Button_Switch_SMD:SW_SPST_B3U-1000P
Changed lines of the file:
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@@
 			)
 		)
-		(property "Footprint" "Connector_USB:USB_C_Receptacle_GCT_USB4110"
+		(property "Footprint" "open-pe:USB_C_Receptacle_GCT_USB4110"
 			(at 203.2 45.72 0)
 			(effects
@@
 			)
 		)
-		(property "Footprint" "Button_Switch_SMD:SW_SPST_B3U-1000P"
+		(property "Footprint" "Button_Switch_SMD:SW_Push_SPST_NO_Alps_SKRK"
 			(at 233.68 74.93 0)
 			(effects
@@
 			(at 233.68 80.01 0)
 			(effects
+				(font
+					(size 1.27 1.27)
+				)
+				(hide yes)
+			)
+		)
+		(property "Footprint_alt" "Button_Switch_SMD:SW_SPST_B3U-1000P"
+			(at 233.68 80.01 0)
+			(effects

Commit message: up
Parts:
- added D5: D_Schottky, Diode_SMD:D_SOD-123, symbol Device:D_Schottky
- C2: value 1uF, 16V -> 22uF, 10V; footprint Capacitor_SMD:C_0805_2012Metric -> Capacitor_SMD:C_0603_1608Metric_Pad1.08x0.95mm_HandSolder; Digikey (none) -> CL10A226MP8NUNE
Connections:
- net +3.3V: now also D5.2 (A)
- net Vusb: now also D5.1 (K)
Other:
- note added: "diode to protect the LDO against reverse current (but we dont have space)"
Changed lines of the file:
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@@
 (kicad_sch
-	(version 20231120)
+	(version 20250114)
 	(generator "eeschema")
-	(generator_version "8.0")
+	(generator_version "9.0")
 	(paper "A4")
+	(text "startup delay (link)"
+		(exclude_from_sim no)
+		(at 26.67 66.04 0)
+		(effects
+			(font
+				(size 1.27 1.27)
+			)
+			(justify left bottom)
+			(href "https://www.espressif.com/sites/default/files/documentation/esp32-s3-wroom-1_wroom-1u_datasheet_en.pdf#page=28")
+		)
+	)
+	(text "diode to protect\nthe LDO against\nreverse current\n(but we dont have space)"
+		(exclude_from_sim no)
+		(at 255.905 111.125 0)
+		(effects
+			(font
+				(size 1.27 1.27)
+			)
+		)
+	)
+	(text "GPIO 1-20 have\nboot glitches,\n18-20 high!"
+		(exclude_from_sim no)
+		(at 58.42 128.27 0)
+		(effects
+			(font
+				(size 1.27 1.27)
+			)
+			(justify left bottom)
+			(href "https://www.espressif.com/sites/default/files/documentation/esp32-s3_datasheet_en.pdf#page=14")
+		)
+	)
+	(text "todo pull up cap?\n"
+		(exclude_from_sim no)
+		(at 184.15 140.97 0)
+		(effects
+			(font
+				(size 1.27 1.27)
+			)
+			(justify left bottom)
+		)
+	)
+	(text "USB Flashing\nhttps://developer.espressif.com/blog/dfu-using-the-native-usb-on-esp32-s2-for-flashing-the-firmware/\n\nUSB DFU (Device Firmware Upgrade)\n\"After connecting and powering the board, we are able to enter in DFU mode by holding BOOT and pressing and releasing the RST (reset) button.\""
+		(exclude_from_sim no)
+		(at 23.114 168.402 0)
+		(effects
+			(font
+				(size 1.27 1.27)
+			)
+			(justify left)
+		)
+	)
 	(junction
 		(at 231.14 128.27)
@@
 	)
 	(junction
+		(at 250.825 125.73)
+		(diameter 0)
+		(color 0 0 0 0)
+	)
+	(junction
 		(at 185.42 93.98)
 		(diameter 0)
@@
 	)
 	(junction
+		(at 255.27 125.73)
+		(diameter 0)
+		(color 0 0 0 0)
+	)
+	(junction
 		(at 228.6 128.27)
 		(diameter 0)
@@
 		(color 0 0 0 0)
 	)
-	(junction
-		(at 255.27 128.27)
-		(diameter 0)
-		(color 0 0 0 0)
-	)
 	(no_connect
 		(at 24.13 135.89)
@@
 	(wire
 		(pts
+			(xy 255.27 125.73) (xy 255.27 129.54)
+		)
+		(stroke
+			(width 0)
+			(type default)
+		)
+	)
+	(wire
+		(pts
 			(xy 115.57 135.89) (xy 116.84 135.89)
 		)
@@
 	(wire
 		(pts
+			(xy 250.825 125.73) (xy 255.27 125.73)
+		)
+		(stroke
+			(width 0)
+			(type default)
+		)
+	)
+	(wire
+		(pts
 			(xy 24.13 63.5) (xy 40.64 63.5)
 		)
@@
 	(wire
 		(pts
-			(xy 247.65 125.73) (xy 247.65 128.27)
+			(xy 69.85 64.77) (xy 69.85 66.04)
 		)
 		(stroke
@@
 	(wire
 		(pts
-			(xy 69.85 64.77) (xy 69.85 66.04)
+			(xy 115.57 113.03) (xy 116.84 113.03)
 		)
 		(stroke
@@
 	(wire
 		(pts
-			(xy 115.57 113.03) (xy 116.84 113.03)
+			(xy 58.42 66.04) (xy 40.64 66.04)
 		)
 		(stroke
@@
 	(wire
 		(pts
-			(xy 58.42 66.04) (xy 40.64 66.04)
+			(xy 236.22 116.84) (xy 228.6 116.84)
 		)
 		(stroke
@@
 	(wire
 		(pts
-			(xy 247.65 128.27) (xy 255.27 128.27)
+			(xy 243.84 116.84) (xy 250.825 116.84)
 		)
 		(stroke
@@
 	(wire
 		(pts
+			(xy 228.6 116.84) (xy 228.6 128.27)
+		)
+		(stroke
+			(width 0)
+			(type default)
+		)
+	)
+	(wire
+		(pts
 			(xy 81.28 64.77) (xy 82.55 64.77)
 		)
@@
 	(wire
 		(pts
-			(xy 255.27 127) (xy 255.27 128.27)
+			(xy 255.27 124.46) (xy 255.27 125.73)
 		)
 		(stroke
@@
 	(wire
 		(pts
-			(xy 133.35 36.83) (xy 135.89 36.83)
+			(xy 250.825 116.84) (xy 250.825 125.73)
 		)
 		(stroke
@@
 	(wire
 		(pts
-			(xy 255.27 128.27) (xy 255.27 129.54)
+			(xy 133.35 36.83) (xy 135.89 36.83)
 		)
 		(stroke
@@
 		)
 	)
-	(text "startup delay (link)"
-		(exclude_from_sim no)
-		(at 26.67 66.04 0)
-		(effects
-			(font
-				(size 1.27 1.27)
-			)
-			(justify left bottom)
-			(href "https://www.espressif.com/sites/default/files/documentation/esp32-s3-wroom-1_wroom-1u_datasheet_en.pdf#page=28")
-		)
-	)
-	(text "GPIO 1-20 have\nboot glitches,\n18-20 high!"
-		(exclude_from_sim no)
-		(at 58.42 128.27 0)
-		(effects
-			(font
-				(size 1.27 1.27)
-			)
-			(justify left bottom)
-			(href "https://www.espressif.com/sites/default/files/documentation/esp32-s3_datasheet_en.pdf#page=14")
-		)
-	)
-	(text "todo pull up cap?\n"
-		(exclude_from_sim no)
-		(at 184.15 140.97 0)
-		(effects
-			(font
-				(size 1.27 1.27)
-			)
-			(justify left bottom)
+	(wire
+		(pts
+			(xy 247.65 125.73) (xy 250.825 125.73)
 		)
-	)
-	(text "USB Flashing\nhttps://developer.espressif.com/blog/dfu-using-the-native-usb-on-esp32-s2-for-flashing-the-firmware/\n\nUSB DFU (Device Firmware Upgrade)\n\"After connecting and powering the board, we are able to enter in DFU mode by holding BOOT and pressing and releasing the RST (reset) button.\""
-		(exclude_from_sim no)
-		(at 23.114 168.402 0)
-		(effects
-			(font
-				(size 1.27 1.27)
-			)
-			(justify left)
+		(stroke
+			(width 0)
+			(type default)
 		)
 	)
@@
 	)
 	(symbol
+		(lib_id "Device:D_Schottky")
+		(at 240.03 116.84 0)
+		(unit 1)
+		(exclude_from_sim yes)
+		(in_bom no)
+		(on_board no)
+		(dnp yes)
+		(fields_autoplaced yes)
+		(property "Reference" "D5"
+			(at 239.7125 110.49 0)
+			(effects
+				(font
+					(size 1.27 1.27)
+				)
+			)
+		)
+		(property "Value" "D_Schottky"
+			(at 239.7125 113.03 0)
+			(effects
+				(font
+					(size 1.27 1.27)
+				)
+			)
+		)
+		(property "Footprint" "Diode_SMD:D_SOD-123"
+			(at 240.03 116.84 0)
+			(effects
+				(font
+					(size 1.27 1.27)
+				)
+				(hide yes)
+			)
+		)
+		(property "Datasheet" "~"
+			(at 240.03 116.84 0)
+			(effects
+				(font
+					(size 1.27 1.27)
+				)
+				(hide yes)
+			)
+		)
+		(property "Description" "Schottky diode"
+			(at 240.03 116.84 0)
+			(effects
+				(font
+					(size 1.27 1.27)
+				)
+				(hide yes)
+			)
+		)
+		(pin "1"
+		)
+		(pin "2"
+		)
+		(instances
+			(project ""
+				(path "/83da95f0-bbf6-49f7-ba45-bd185bc958bc"
+					(reference "D5")
+					(unit 1)
+				)
+			)
+		)
+	)
+	(symbol
 		(lib_id "Connector:USB_C_Plug_USB2.0")
 		(at 203.2 41.91 270)
@@
 	(symbol
 		(lib_id "power:+3.3V")
-		(at 255.27 127 0)
+		(at 255.27 124.46 0)
 		(mirror y)
 		(unit 1)
@@
 		(dnp no)
 		(property "Reference" "#PWR012"
-			(at 255.27 130.81 0)
+			(at 255.27 128.27 0)
 			(effects
 				(font
@@
 		)
 		(property "Value" "+3.3V"
-			(at 262.636 126.492 0)
+			(at 262.636 123.952 0)
 			(effects
 				(font
@@
 		)
 		(property "Footprint" ""
-			(at 255.27 127 0)
+			(at 255.27 124.46 0)
 			(effects
 				(font
@@
 		)
 		(property "Datasheet" ""
-			(at 255.27 127 0)
+			(at 255.27 124.46 0)
 			(effects
 				(font
@@
 		)
 		(property "Description" ""
-			(at 255.27 127 0)
+			(at 255.27 124.46 0)
 			(effects
 				(font
@@
 		(at 214.63 128.27 180)
 		(unit 1)
-		(exclude_from_sim no)
+		(exclude_from_sim yes)
 		(in_bom no)
 		(on_board no)
@@
 			)
 		)
-		(property "Value" "1uF, 16V"
+		(property "Value" "22uF, 10V"
 			(at 249.936 130.81 0)
 			(effects
@@
 			)
 		)
-		(property "Footprint" "Capacitor_SMD:C_0805_2012Metric"
+		(property "Footprint" "Capacitor_SMD:C_0603_1608Metric_Pad1.08x0.95mm_HandSolder"
 			(at 255.27 132.08 0)
 			(effects
@@
 			)
 		)
+		(property "Digikey" "CL10A226MP8NUNE"
+			(at 255.27 132.08 0)
+			(effects
+				(font
+					(size 1.27 1.27)
+				)
+				(hide yes)
+			)
+		)
 		(pin "1"
 		)
@@
 		)
 	)
+	(embedded_fonts no)
 )
